Commit message: update

File: wheelmecanum.urdf (robot description, URDF)
Before this commit: robot wheel, 13 links, 12 joints
Links:
- link mcn1: geometry collision mesh filename=/home/samet/Desktop/robomaster-stl-files/wheels/mecanumroll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 scale=0.002 0.002 0.002; visual mesh filename=/home/samet/Desktop/robomaster-stl-files/wheels/mecanumroll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 scale=0.002 0.002 0.002
- link mcn10: geometry collision mesh filename=/home/samet/Desktop/robomaster-stl-files/wheels/mecanumroll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 scale=0.002 0.002 0.002; visual mesh filename=/home/samet/Desktop/robomaster-stl-files/wheels/mecanumroll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 scale=0.002 0.002 0.002
- link mcn11: geometry collision mesh filename=/home/samet/Desktop/robomaster-stl-files/wheels/mecanumroll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 scale=0.002 0.002 0.002; visual mesh filename=/home/samet/Desktop/robomaster-stl-files/wheels/mecanumroll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 scale=0.002 0.002 0.002
- link mcn12: geometry collision mesh filename=/home/samet/Desktop/robomaster-stl-files/wheels/mecanumroll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 scale=0.002 0.002 0.002; visual mesh filename=/home/samet/Desktop/robomaster-stl-files/wheels/mecanumroll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 scale=0.002 0.002 0.002
- link mcn2: geometry collision mesh filename=/home/samet/Desktop/robomaster-stl-files/wheels/mecanumroll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 scale=0.002 0.002 0.002; visual mesh filename=/home/samet/Desktop/robomaster-stl-files/wheels/mecanumroll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 scale=0.002 0.002 0.002
- link mcn3: geometry collision mesh filename=/home/samet/Desktop/robomaster-stl-files/wheels/mecanumroll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 scale=0.002 0.002 0.002; visual mesh filename=/home/samet/Desktop/robomaster-stl-files/wheels/mecanumroll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 scale=0.002 0.002 0.002
- link mcn4: geometry collision mesh filename=/home/samet/Desktop/robomaster-stl-files/wheels/mecanumroll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 scale=0.002 0.002 0.002; visual mesh filename=/home/samet/Desktop/robomaster-stl-files/wheels/mecanumroll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 scale=0.002 0.002 0.002
- link mcn5: geometry collision mesh filename=/home/samet/Desktop/robomaster-stl-files/wheels/mecanumroll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 scale=0.002 0.002 0.002; visual mesh filename=/home/samet/Desktop/robomaster-stl-files/wheels/mecanumroll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 scale=0.002 0.002 0.002
- link mcn6: geometry collision mesh filename=/home/samet/Desktop/robomaster-stl-files/wheels/mecanumroll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 scale=0.002 0.002 0.002; visual mesh filename=/home/samet/Desktop/robomaster-stl-files/wheels/mecanumroll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 scale=0.002 0.002 0.002
- link mcn7: geometry collision mesh filename=/home/samet/Desktop/robomaster-stl-files/wheels/mecanumroll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 scale=0.002 0.002 0.002; visual mesh filename=/home/samet/Desktop/robomaster-stl-files/wheels/mecanumroll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 scale=0.002 0.002 0.002
- link mcn8: geometry collision mesh filename=/home/samet/Desktop/robomaster-stl-files/wheels/mecanumroll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 scale=0.002 0.002 0.002; visual mesh filename=/home/samet/Desktop/robomaster-stl-files/wheels/mecanumroll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 scale=0.002 0.002 0.002
- link mcn9: geometry collision mesh filename=/home/samet/Desktop/robomaster-stl-files/wheels/mecanumroll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 scale=0.002 0.002 0.002; visual mesh filename=/home/samet/Desktop/robomaster-stl-files/wheels/mecanumroll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 scale=0.002 0.002 0.002
