Commit message: update

File: kodlar/arkatekerler/omnihazirL.xacro (robot description, xacro)
@@ -11,5 +11,5 @@
         <origin xyz="0 0 0" rpy="0 0 0"/>
         <geometry>
-          <mesh filename="file:///home/samet/Desktop/isaac_robomaster/meshes/stl/mecanummain.stl" scale="0.002 0.002 0.002"/>
+          <mesh filename="/home/samet/Desktop/isaac_robomaster/meshes/stl/mecanummain.stl" scale="0.002 0.002 0.002"/>
         </geometry>
       </visual>
@@ -30,5 +30,5 @@
         <origin xyz="0 0 0" rpy="0 0 0"/>
         <geometry>
-          <mesh filename="file:///home/samet/Desktop/isaac_robomaster/meshes/stl/mecanumroller.stl" scale="0.002 0.002 0.002"/>
+          <mesh filename="/home/samet/Desktop/isaac_robomaster/meshes/stl/mecanumroller.stl" scale="0.002 0.002 0.002"/>
         </geometry>
       </visual>
@@ -36,5 +36,5 @@
         <origin xyz="0 0 0" rpy="0 0 0"/>
         <geometry>
-          <mesh filename="file:///home/samet/Desktop/isaac_robomaster/meshes/stl/mecanumroller.stl" scale="0.002 0.002 0.002"/>
+          <mesh filename="/home/samet/Desktop/isaac_robomaster/meshes/stl/mecanumroller.stl" scale="0.002 0.002 0.002"/>
         </geometry>
       </collision>
@@ -49,5 +49,5 @@
         <origin xyz="0 0 0" rpy="0 0 0"/>
         <geometry>
-          <mesh filename="file:///home/samet/Desktop/isaac_robomaster/meshes/stl/mecanumroller.stl" scale="0.002 0.002 0.002"/>
+          <mesh filename="/home/samet/Desktop/isaac_robomaster/meshes/stl/mecanumroller.stl" scale="0.002 0.002 0.002"/>
         </geometry>
       </visual>
@@ -55,5 +55,5 @@
         <origin xyz="0 0 0" rpy="0 0 0"/>
         <geometry>
-          <mesh filename="file:///home/samet/Desktop/isaac_robomaster/meshes/stl/mecanumroller.stl" scale="0.002 0.002 0.002"/>
+          <mesh filename="/home/samet/Desktop/isaac_robomaster/meshes/stl/mecanumroller.stl" scale="0.002 0.002 0.002"/>
         </geometry>
       </collision>
@@ -68,5 +68,5 @@
         <origin xyz="0 0 0" rpy="0 0 0"/>
         <geometry>
-          <mesh filename="file:///home/samet/Desktop/isaac_robomaster/meshes/stl/mecanumroller.stl" scale="0.002 0.002 0.002"/>
+          <mesh filename="/home/samet/Desktop/isaac_robomaster/meshes/stl/mecanumroller.stl" scale="0.002 0.002 0.002"/>
         </geometry>
       </visual>
@@ -74,5 +74,5 @@
         <origin xyz="0 0 0" rpy="0 0 0"/>
         <geometry>
-          <mesh filename="file:///home/samet/Desktop/isaac_robomaster/meshes/stl/mecanumroller.stl" scale="0.002 0.002 0.002"/>
+          <mesh filename="/home/samet/Desktop/isaac_robomaster/meshes/stl/mecanumroller.stl" scale="0.002 0.002 0.002"/>
         </geometry>
       </collision>
@@ -87,5 +87,5 @@
         <origin xyz="0 0 0" rpy="0 0 0"/>
         <geometry>
-          <mesh filename="file:///home/samet/Desktop/isaac_robomaster/meshes/stl/mecanumroller.stl" scale="0.002 0.002 0.002"/>
+          <mesh filename="/home/samet/Desktop/isaac_robomaster/meshes/stl/mecanumroller.stl" scale="0.002 0.002 0.002"/>
         </geometry>
       </visual>
@@ -93,5 +93,5 @@
         <origin xyz="0 0 0" rpy="0 0 0"/>
         <geometry>
-          <mesh filename="file:///home/samet/Desktop/isaac_robomaster/meshes/stl/mecanumroller.stl" scale="0.002 0.002 0.002"/>
+          <mesh filename="/home/samet/Desktop/isaac_robomaster/meshes/stl/mecanumroller.stl" scale="0.002 0.002 0.002"/>
         </geometry>
       </collision>
@@ -106,5 +106,5 @@
         <origin xyz="0 0 0" rpy="0 0 0"/>
         <geometry>
-          <mesh filename="file:///home/samet/Desktop/isaac_robomaster/meshes/stl/mecanumroller.stl" scale="0.002 0.002 0.002"/>
+          <mesh filename="/home/samet/Desktop/isaac_robomaster/meshes/stl/mecanumroller.stl" scale="0.002 0.002 0.002"/>
         </geometry>
       </visual>
@@ -112,5 +112,5 @@
         <origin xyz="0 0 0" rpy="0 0 0"/>
         <geometry>
-          <mesh filename="file:///home/samet/Desktop/isaac_robomaster/meshes/stl/mecanumroller.stl" scale="0.002 0.002 0.002"/>
+          <mesh filename="/home/samet/Desktop/isaac_robomaster/meshes/stl/mecanumroller.stl" scale="0.002 0.002 0.002"/>
         </geometry>
       </collision>
@@ -125,5 +125,5 @@
         <origin xyz="0 0 0" rpy="0 0 0"/>
         <geometry>
-          <mesh filename="file:///home/samet/Desktop/isaac_robomaster/meshes/stl/mecanumroller.stl" scale="0.002 0.002 0.002"/>
+          <mesh filename="/home/samet/Desktop/isaac_robomaster/meshes/stl/mecanumroller.stl" scale="0.002 0.002 0.002"/>
         </geometry>
       </visual>
@@ -131,5 +131,5 @@
         <origin xyz="0 0 0" rpy="0 0 0"/>
         <geometry>
-          <mesh filename="file:///home/samet/Desktop/isaac_robomaster/meshes/stl/mecanumroller.stl" scale="0.002 0.002 0.002"/>
+          <mesh filename="/home/samet/Desktop/isaac_robomaster/meshes/stl/mecanumroller.stl" scale="0.002 0.002 0.002"/>
         </geometry>
       </collision>
@@ -144,5 +144,5 @@
         <origin xyz="0 0 0" rpy="0 0 0"/>
         <geometry>
-          <mesh filename="file:///home/samet/Desktop/isaac_robomaster/meshes/stl/mecanumroller.stl" scale="0.002 0.002 0.002"/>
+          <mesh filename="/home/samet/Desktop/isaac_robomaster/meshes/stl/mecanumroller.stl" scale="0.002 0.002 0.002"/>
         </geometry>
       </visual>
@@ -150,5 +150,5 @@
         <origin xyz="0 0 0" rpy="0 0 0"/>
         <geometry>
-          <mesh filename="file:///home/samet/Desktop/isaac_robomaster/meshes/stl/mecanumroller.stl" scale="0.002 0.002 0.002"/>
+          <mesh filename="/home/samet/Desktop/isaac_robomaster/meshes/stl/mecanumroller.stl" scale="0.002 0.002 0.002"/>
         </geometry>
       </collision>
@@ -163,5 +163,5 @@
         <origin xyz="0 0 0" rpy="0 0 0"/>
         <geometry>
-          <mesh filename="file:///home/samet/Desktop/isaac_robomaster/meshes/stl/mecanumroller.stl" scale="0.002 0.002 0.002"/>
+          <mesh filename="/home/samet/Desktop/isaac_robomaster/meshes/stl/mecanumroller.stl" scale="0.002 0.002 0.002"/>
         </geometry>
       </visual>
@@ -169,5 +169,5 @@
         <origin xyz="0 0 0" rpy="0 0 0"/>
         <geometry>
-          <mesh filename="file:///home/samet/Desktop/isaac_robomaster/meshes/stl/mecanumroller.stl" scale="0.002 0.002 0.002"/>
+          <mesh filename="/home/samet/Desktop/isaac_robomaster/meshes/stl/mecanumroller.stl" scale="0.002 0.002 0.002"/>
         </geometry>
       </collision>
@@ -182,5 +182,5 @@
         <origin xyz="0 0 0" rpy="0 0 0"/>
         <geometry>
-          <mesh filename="file:///home/samet/Desktop/isaac_robomaster/meshes/stl/mecanumroller.stl" scale="0.002 0.002 0.002"/>
+          <mesh filename="/home/samet/Desktop/isaac_robomaster/meshes/stl/mecanumroller.stl" scale="0.002 0.002 0.002"/>
         </geometry>
       </visual>
@@ -188,5 +188,5 @@
         <origin xyz="0 0 0" rpy="0 0 0"/>
         <geometry>
-          <mesh filename="file:///home/samet/Desktop/isaac_robomaster/meshes/stl/mecanumroller.stl" scale="0.002 0.002 0.002"/>
+          <mesh filename="/home/samet/Desktop/isaac_robomaster/meshes/stl/mecanumroller.stl" scale="0.002 0.002 0.002"/>
         </geometry>
       </collision>
@@ -201,5 +201,5 @@
         <origin xyz="0 0 0" rpy="0 0 0"/>
         <geometry>
-          <mesh filename="file:///home/samet/Desktop/isaac_robomaster/meshes/stl/mecanumroller.stl" scale="0.002 0.002 0.002"/>
+          <mesh filename="/home/samet/Desktop/isaac_robomaster/meshes/stl/mecanumroller.stl" scale="0.002 0.002 0.002"/>
         </geometry>
       </visual>
@@ -207,5 +207,5 @@
         <origin xyz="0 0 0" rpy="0 0 0"/>
         <geometry>
-          <mesh filename="file:///home/samet/Desktop/isaac_robomaster/meshes/stl/mecanumroller.stl" scale="0.002 0.002 0.002"/>
+          <mesh filename="/home/samet/Desktop/isaac_robomaster/meshes/stl/mecanumroller.stl" scale="0.002 0.002 0.002"/>
         </geometry>
       </collision>
@@ -220,5 +220,5 @@
         <origin xyz="0 0 0" rpy="0 0 0"/>
         <geometry>
-          <mesh filename="file:///home/samet/Desktop/isaac_robomaster/meshes/stl/mecanumroller.stl" scale="0.002 0.002 0.002"/>
+          <mesh filename="/home/samet/Desktop/isaac_robomaster/meshes/stl/mecanumroller.stl" scale="0.002 0.002 0.002"/>
         </geometry>
       </visual>
@@ -226,5 +226,5 @@
         <origin xyz="0 0 0" rpy="0 0 0"/>
         <geometry>
-          <mesh filename="file:///home/samet/Desktop/isaac_robomaster/meshes/stl/mecanumroller.stl" scale="0.002 0.002 0.002"/>
+          <mesh filename="/home/samet/Desktop/isaac_robomaster/meshes/stl/mecanumroller.stl" scale="0.002 0.002 0.002"/>
         </geometry>
       </collision>
@@ -239,5 +239,5 @@
         <origin xyz="0 0 0" rpy="0 0 0"/>
         <geometry>
-          <mesh filename="file:///home/samet/Desktop/isaac_robomaster/meshes/stl/mecanumroller.stl" scale="0.002 0.002 0.002"/>
+          <mesh filename="/home/samet/Desktop/isaac_robomaster/meshes/stl/mecanumroller.stl" scale="0.002 0.002 0.002"/>
         </geometry>
       </visual>
@@ -245,5 +245,5 @@
         <origin xyz="0 0 0" rpy="0 0 0"/>
         <geometry>
-          <mesh filename="file:///home/samet/Desktop/isaac_robomaster/meshes/stl/mecanumroller.stl" scale="0.002 0.002 0.002"/>
+          <mesh filename="/home/samet/Desktop/isaac_robomaster/meshes/stl/mecanumroller.stl" scale="0.002 0.002 0.002"/>
         </geometry>
       </collision>
