Commit message: update

File: kodlar/arkatekerler/omnihazirR.xacro (robot description, xacro)
@@ -1,6 +1,6 @@
 <?xml version="1.0"?>
 <robot xmlns:xacro="http://www.ros.org/wiki/xacro" >
-<xacro:macro name="leko">
-<link name="base_link">
+<xacro:macro name="leko2">
+<link name="base_link2">
       <inertial>
         <origin xyz="0 0 0" rpy="0 0 0"/>
@@ -8,11 +8,11 @@
         <inertia ixx="0.1" ixy="0" ixz="0" iyy="0.1" iyz="0" izz="0.1"/>
       </inertial>
-      <visual name="visual_0_base_link">
-        <origin xyz="0 0 0" rpy="0 0 0"/>
-        <geometry>
-          <mesh filename="file:///home/samet/Desktop/isaac_robomaster/meshes/stl/mecanummain.stl" scale="0.002 0.002 0.002"/>
-        </geometry>
-      </visual>
-      <collision name="collision_0_base_link">
+      <visual>
+        <origin xyz="0 0 0" rpy="0 0 0"/>
+        <geometry>
+          <mesh filename="/home/samet/Desktop/isaac_robomaster/meshes/stl/mecanummain.stl" scale="0.002 0.002 0.002"/>
+        </geometry>
+      </visual>
+      <collision>
         <origin xyz="0 0 0" rpy="0 0 0"/>
         <geometry>
@@ -21,302 +21,302 @@
       </collision>
     </link>
-    <link name="mcn1">
-      <inertial>
-        <origin xyz="0 0 0" rpy="0 0 0"/>
-        <mass value="0.03"/>
-        <inertia ixx="0.1" ixy="0" ixz="0" iyy="0.1" iyz="0" izz="0.1"/>
-      </inertial>
-      <visual name="visual_0_mcn1">
-        <origin xyz="0 0 0" rpy="0 0 0"/>
-        <geometry>
-          <mesh filename="file:///home/samet/Desktop/isaac_robomaster/meshes/stl/mecanumroller.stl" scale="0.002 0.002 0.002"/>
-        </geometry>
-      </visual>
-      <collision name="collision_0_mcn1">
-        <origin xyz="0 0 0" rpy="0 0 0"/>
-        <geometry>
-          <mesh filename="file:///home/samet/Desktop/isaac_robomaster/meshes/stl/mecanumroller.stl" scale="0.002 0.002 0.002"/>
-        </geometry>
-      </collision>
-    </link>
-    <link name="mcn10">
-      <inertial>
-        <origin xyz="0 0 0" rpy="0 0 0"/>
-        <mass value="0.03"/>
-        <inertia ixx="0.1" ixy="0" ixz="0" iyy="0.1" iyz="0" izz="0.1"/>
-      </inertial>
-      <visual name="visual_0_mcn10">
-        <origin xyz="0 0 0" rpy="0 0 0"/>
-        <geometry>
-          <mesh filename="file:///home/samet/Desktop/isaac_robomaster/meshes/stl/mecanumroller.stl" scale="0.002 0.002 0.002"/>
-        </geometry>
-      </visual>
-      <collision name="collision_0_mcn10">
-        <origin xyz="0 0 0" rpy="0 0 0"/>
-        <geometry>
-          <mesh filename="file:///home/samet/Desktop/isaac_robomaster/meshes/stl/mecanumroller.stl" scale="0.002 0.002 0.002"/>
-        </geometry>
-      </collision>
-    </link>
-    <link name="mcn11">
-      <inertial>
-        <origin xyz="0 0 0" rpy="0 0 0"/>
-        <mass value="0.03"/>
-        <inertia ixx="0.1" ixy="0" ixz="0" iyy="0.1" iyz="0" izz="0.1"/>
-      </inertial>
-      <visual name="visual_0_mcn11">
-        <origin xyz="0 0 0" rpy="0 0 0"/>
-        <geometry>
-          <mesh filename="file:///home/samet/Desktop/isaac_robomaster/meshes/stl/mecanumroller.stl" scale="0.002 0.002 0.002"/>
-        </geometry>
-      </visual>
-      <collision name="collision_0_mcn11">
-        <origin xyz="0 0 0" rpy="0 0 0"/>
-        <geometry>
-          <mesh filename="file:///home/samet/Desktop/isaac_robomaster/meshes/stl/mecanumroller.stl" scale="0.002 0.002 0.002"/>
-        </geometry>
-      </collision>
-    </link>
-    <link name="mcn12">
-      <inertial>
-        <origin xyz="0 0 0" rpy="0 0 0"/>
-        <mass value="0.03"/>
-        <inertia ixx="0.1" ixy="0" ixz="0" iyy="0.1" iyz="0" izz="0.1"/>
-      </inertial>
-      <visual name="visual_0_mcn12">
-        <origin xyz="0 0 0" rpy="0 0 0"/>
-        <geometry>
-          <mesh filename="file:///home/samet/Desktop/isaac_robomaster/meshes/stl/mecanumroller.stl" scale="0.002 0.002 0.002"/>
-        </geometry>
-      </visual>
-      <collision name="collision_0_mcn12">
-        <origin xyz="0 0 0" rpy="0 0 0"/>
-        <geometry>
-          <mesh filename="file:///home/samet/Desktop/isaac_robomaster/meshes/stl/mecanumroller.stl" scale="0.002 0.002 0.002"/>
-        </geometry>
-      </collision>
-    </link>
-    <link name="mcn2">
-      <inertial>
-        <origin xyz="0 0 0" rpy="0 0 0"/>
-        <mass value="0.03"/>
-        <inertia ixx="0.1" ixy="0" ixz="0" iyy="0.1" iyz="0" izz="0.1"/>
-      </inertial>
-      <visual name="visual_0_mcn2">
-        <origin xyz="0 0 0" rpy="0 0 0"/>
-        <geometry>
-          <mesh filename="file:///home/samet/Desktop/isaac_robomaster/meshes/stl/mecanumroller.stl" scale="0.002 0.002 0.002"/>
-        </geometry>
-      </visual>
-      <collision name="collision_0_mcn2">
-        <origin xyz="0 0 0" rpy="0 0 0"/>
-        <geometry>
-          <mesh filename="file:///home/samet/Desktop/isaac_robomaster/meshes/stl/mecanumroller.stl" scale="0.002 0.002 0.002"/>
-        </geometry>
-      </collision>
-    </link>
-    <link name="mcn3">
-      <inertial>
-        <origin xyz="0 0 0" rpy="0 0 0"/>
-        <mass value="0.03"/>
-        <inertia ixx="0.1" ixy="0" ixz="0" iyy="0.1" iyz="0" izz="0.1"/>
-      </inertial>
-      <visual name="visual_0_mcn3">
-        <origin xyz="0 0 0" rpy="0 0 0"/>
-        <geometry>
-          <mesh filename="file:///home/samet/Desktop/isaac_robomaster/meshes/stl/mecanumroller.stl" scale="0.002 0.002 0.002"/>
-        </geometry>
-      </visual>
-      <collision name="collision_0_mcn3">
-        <origin xyz="0 0 0" rpy="0 0 0"/>
-        <geometry>
-          <mesh filename="file:///home/samet/Desktop/isaac_robomaster/meshes/stl/mecanumroller.stl" scale="0.002 0.002 0.002"/>
-        </geometry>
-      </collision>
-    </link>
-    <link name="mcn4">
-      <inertial>
-        <origin xyz="0 0 0" rpy="0 0 0"/>
-        <mass value="0.03"/>
-        <inertia ixx="0.1" ixy="0" ixz="0" iyy="0.1" iyz="0" izz="0.1"/>
-      </inertial>
-      <visual name="visual_0_mcn4">
-        <origin xyz="0 0 0" rpy="0 0 0"/>
-        <geometry>
-          <mesh filename="file:///home/samet/Desktop/isaac_robomaster/meshes/stl/mecanumroller.stl" scale="0.002 0.002 0.002"/>
-        </geometry>
-      </visual>
-      <collision name="collision_0_mcn4">
-        <origin xyz="0 0 0" rpy="0 0 0"/>
-        <geometry>
-          <mesh filename="file:///home/samet/Desktop/isaac_robomaster/meshes/stl/mecanumroller.stl" scale="0.002 0.002 0.002"/>
-        </geometry>
-      </collision>
-    </link>
-    <link name="mcn5">
-      <inertial>
-        <origin xyz="0 0 0" rpy="0 0 0"/>
-        <mass value="0.03"/>
-        <inertia ixx="0.1" ixy="0" ixz="0" iyy="0.1" iyz="0" izz="0.1"/>
-      </inertial>
-      <visual name="visual_0_mcn5">
-        <origin xyz="0 0 0" rpy="0 0 0"/>
-        <geometry>
-          <mesh filename="file:///home/samet/Desktop/isaac_robomaster/meshes/stl/mecanumroller.stl" scale="0.002 0.002 0.002"/>
-        </geometry>
-      </visual>
-      <collision name="collision_0_mcn5">
-        <origin xyz="0 0 0" rpy="0 0 0"/>
-        <geometry>
-          <mesh filename="file:///home/samet/Desktop/isaac_robomaster/meshes/stl/mecanumroller.stl" scale="0.002 0.002 0.002"/>
-        </geometry>
-      </collision>
-    </link>
-    <link name="mcn6">
-      <inertial>
-        <origin xyz="0 0 0" rpy="0 0 0"/>
-        <mass value="0.03"/>
-        <inertia ixx="0.1" ixy="0" ixz="0" iyy="0.1" iyz="0" izz="0.1"/>
-      </inertial>
-      <visual name="visual_0_mcn6">
-        <origin xyz="0 0 0" rpy="0 0 0"/>
-        <geometry>
-          <mesh filename="file:///home/samet/Desktop/isaac_robomaster/meshes/stl/mecanumroller.stl" scale="0.002 0.002 0.002"/>
-        </geometry>
-      </visual>
-      <collision name="collision_0_mcn6">
-        <origin xyz="0 0 0" rpy="0 0 0"/>
-        <geometry>
-          <mesh filename="file:///home/samet/Desktop/isaac_robomaster/meshes/stl/mecanumroller.stl" scale="0.002 0.002 0.002"/>
-        </geometry>
-      </collision>
-    </link>
-    <link name="mcn7">
-      <inertial>
-        <origin xyz="0 0 0" rpy="0 0 0"/>
-        <mass value="0.03"/>
-        <inertia ixx="0.1" ixy="0" ixz="0" iyy="0.1" iyz="0" izz="0.1"/>
-      </inertial>
-      <visual name="visual_0_mcn7">
-        <origin xyz="0 0 0" rpy="0 0 0"/>
-        <geometry>
-          <mesh filename="file:///home/samet/Desktop/isaac_robomaster/meshes/stl/mecanumroller.stl" scale="0.002 0.002 0.002"/>
-        </geometry>
-      </visual>
-      <collision name="collision_0_mcn7">
-        <origin xyz="0 0 0" rpy="0 0 0"/>
-        <geometry>
-          <mesh filename="file:///home/samet/Desktop/isaac_robomaster/meshes/stl/mecanumroller.stl" scale="0.002 0.002 0.002"/>
-        </geometry>
-      </collision>
-    </link>
-    <link name="mcn8">
-      <inertial>
-        <origin xyz="0 0 0" rpy="0 0 0"/>
-        <mass value="0.03"/>
-        <inertia ixx="0.1" ixy="0" ixz="0" iyy="0.1" iyz="0" izz="0.1"/>
-      </inertial>
-      <visual name="visual_0_mcn8">
-        <origin xyz="0 0 0" rpy="0 0 0"/>
-        <geometry>
-          <mesh filename="file:///home/samet/Desktop/isaac_robomaster/meshes/stl/mecanumroller.stl" scale="0.002 0.002 0.002"/>
-        </geometry>
-      </visual>
-      <collision name="collision_0_mcn8">
-        <origin xyz="0 0 0" rpy="0 0 0"/>
-        <geometry>
-          <mesh filename="file:///home/samet/Desktop/isaac_robomaster/meshes/stl/mecanumroller.stl" scale="0.002 0.002 0.002"/>
-        </geometry>
-      </collision>
-    </link>
-    <link name="mcn9">
-      <inertial>
-        <origin xyz="0 0 0" rpy="0 0 0"/>
-        <mass value="0.03"/>
-        <inertia ixx="0.1" ixy="0" ixz="0" iyy="0.1" iyz="0" izz="0.1"/>
-      </inertial>
-      <visual name="visual_0_mcn9">
-        <origin xyz="0 0 0" rpy="0 0 0"/>
-        <geometry>
-          <mesh filename="file:///home/samet/Desktop/isaac_robomaster/meshes/stl/mecanumroller.stl" scale="0.002 0.002 0.002"/>
-        </geometry>
-      </visual>
-      <collision name="collision_0_mcn9">
-        <origin xyz="0 0 0" rpy="0 0 0"/>
-        <geometry>
-          <mesh filename="file:///home/samet/Desktop/isaac_robomaster/meshes/stl/mecanumroller.stl" scale="0.002 0.002 0.002"/>
-        </geometry>
-      </collision>
-    </link>
-    <joint name="joint1" type="continuous">
+    <link name="mcnN1">
+      <inertial>
+        <origin xyz="0 0 0" rpy="0 0 0"/>
+        <mass value="0.03"/>
+        <inertia ixx="0.1" ixy="0" ixz="0" iyy="0.1" iyz="0" izz="0.1"/>
+      </inertial>
+      <visual>
+        <origin xyz="0 0 0" rpy="0 0 0"/>
+        <geometry>
+          <mesh filename="/home/samet/Desktop/isaac_robomaster/meshes/stl/mecanumroller.stl" scale="0.002 0.002 0.002"/>
+        </geometry>
+      </visual>
+      <collision>
+        <origin xyz="0 0 0" rpy="0 0 0"/>
+        <geometry>
+          <mesh filename="/home/samet/Desktop/isaac_robomaster/meshes/stl/mecanumroller.stl" scale="0.002 0.002 0.002"/>
+        </geometry>
+      </collision>
+    </link>
+    <link name="mcnN10">
+      <inertial>
+        <origin xyz="0 0 0" rpy="0 0 0"/>
+        <mass value="0.03"/>
+        <inertia ixx="0.1" ixy="0" ixz="0" iyy="0.1" iyz="0" izz="0.1"/>
+      </inertial>
+      <visual>
+        <origin xyz="0 0 0" rpy="0 0 0"/>
+        <geometry>
+          <mesh filename="/home/samet/Desktop/isaac_robomaster/meshes/stl/mecanumroller.stl" scale="0.002 0.002 0.002"/>
+        </geometry>
+      </visual>
+      <collision>
+        <origin xyz="0 0 0" rpy="0 0 0"/>
+        <geometry>
+          <mesh filename="/home/samet/Desktop/isaac_robomaster/meshes/stl/mecanumroller.stl" scale="0.002 0.002 0.002"/>
+        </geometry>
+      </collision>
+    </link>
+    <link name="mcnN11">
+      <inertial>
+        <origin xyz="0 0 0" rpy="0 0 0"/>
+        <mass value="0.03"/>
+        <inertia ixx="0.1" ixy="0" ixz="0" iyy="0.1" iyz="0" izz="0.1"/>
+      </inertial>
+      <visual>
+        <origin xyz="0 0 0" rpy="0 0 0"/>
+        <geometry>
+          <mesh filename="/home/samet/Desktop/isaac_robomaster/meshes/stl/mecanumroller.stl" scale="0.002 0.002 0.002"/>
+        </geometry>
+      </visual>
+      <collision>
+        <origin xyz="0 0 0" rpy="0 0 0"/>
+        <geometry>
+          <mesh filename="/home/samet/Desktop/isaac_robomaster/meshes/stl/mecanumroller.stl" scale="0.002 0.002 0.002"/>
+        </geometry>
+      </collision>
+    </link>
+    <link name="mcnN12">
+      <inertial>
+        <origin xyz="0 0 0" rpy="0 0 0"/>
+        <mass value="0.03"/>
+        <inertia ixx="0.1" ixy="0" ixz="0" iyy="0.1" iyz="0" izz="0.1"/>
+      </inertial>
+      <visual>
+        <origin xyz="0 0 0" rpy="0 0 0"/>
+        <geometry>
+          <mesh filename="/home/samet/Desktop/isaac_robomaster/meshes/stl/mecanumroller.stl" scale="0.002 0.002 0.002"/>
+        </geometry>
+      </visual>
+      <collision>
+        <origin xyz="0 0 0" rpy="0 0 0"/>
+        <geometry>
+          <mesh filename="/home/samet/Desktop/isaac_robomaster/meshes/stl/mecanumroller.stl" scale="0.002 0.002 0.002"/>
+        </geometry>
+      </collision>
+    </link>
+    <link name="mcnN2">
+      <inertial>
+        <origin xyz="0 0 0" rpy="0 0 0"/>
+        <mass value="0.03"/>
+        <inertia ixx="0.1" ixy="0" ixz="0" iyy="0.1" iyz="0" izz="0.1"/>
+      </inertial>
+      <visual>
+        <origin xyz="0 0 0" rpy="0 0 0"/>
+        <geometry>
+          <mesh filename="/home/samet/Desktop/isaac_robomaster/meshes/stl/mecanumroller.stl" scale="0.002 0.002 0.002"/>
+        </geometry>
+      </visual>
+      <collision>
+        <origin xyz="0 0 0" rpy="0 0 0"/>
+        <geometry>
+          <mesh filename="/home/samet/Desktop/isaac_robomaster/meshes/stl/mecanumroller.stl" scale="0.002 0.002 0.002"/>
+        </geometry>
+      </collision>
+    </link>
+    <link name="mcnN3">
+      <inertial>
+        <origin xyz="0 0 0" rpy="0 0 0"/>
+        <mass value="0.03"/>
+        <inertia ixx="0.1" ixy="0" ixz="0" iyy="0.1" iyz="0" izz="0.1"/>
+      </inertial>
+      <visual>
+        <origin xyz="0 0 0" rpy="0 0 0"/>
+        <geometry>
+          <mesh filename="/home/samet/Desktop/isaac_robomaster/meshes/stl/mecanumroller.stl" scale="0.002 0.002 0.002"/>
+        </geometry>
+      </visual>
+      <collision>
+        <origin xyz="0 0 0" rpy="0 0 0"/>
+        <geometry>
+          <mesh filename="/home/samet/Desktop/isaac_robomaster/meshes/stl/mecanumroller.stl" scale="0.002 0.002 0.002"/>
+        </geometry>
+      </collision>
+    </link>
+    <link name="mcnN4">
+      <inertial>
+        <origin xyz="0 0 0" rpy="0 0 0"/>
+        <mass value="0.03"/>
+        <inertia ixx="0.1" ixy="0" ixz="0" iyy="0.1" iyz="0" izz="0.1"/>
+      </inertial>
+      <visual>
+        <origin xyz="0 0 0" rpy="0 0 0"/>
+        <geometry>
+          <mesh filename="/home/samet/Desktop/isaac_robomaster/meshes/stl/mecanumroller.stl" scale="0.002 0.002 0.002"/>
+        </geometry>
+      </visual>
+      <collision>
+        <origin xyz="0 0 0" rpy="0 0 0"/>
+        <geometry>
+          <mesh filename="/home/samet/Desktop/isaac_robomaster/meshes/stl/mecanumroller.stl" scale="0.002 0.002 0.002"/>
+        </geometry>
+      </collision>
+    </link>
+    <link name="mcnN5">
+      <inertial>
+        <origin xyz="0 0 0" rpy="0 0 0"/>
+        <mass value="0.03"/>
+        <inertia ixx="0.1" ixy="0" ixz="0" iyy="0.1" iyz="0" izz="0.1"/>
+      </inertial>
+      <visual>
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
File: kodlar/chasishazir.xacro (robot description, xacro)
@@ -1,8 +1,9 @@
 <?xml version="1.0"?>
-<robot name="lqkoooo" xmlns:xacro="http://www.ros.org/wiki/xacro" >
-<link name="base_link">
+<robot  xmlns:xacro="http://www.ros.org/wiki/xacro" >
+<xacro:macro name="chasis">
+<link name="basee_link">
 <visual>
 <geometry>
-    <cylinder radius="0.2" length="0.1"/>
+    <mesh filename="/home/samet/Desktop/robomaster-stl-files/wheels/base_link_centered.stl" scale="0.002 0.002 0.002"/>
 </geometry>
 <origin xyz="0 0 0" rpy="0 0 0"/>
@@ -10,5 +11,5 @@
 <collision>
 <geometry>
-    <cylinder radius="0.2" length="0.1"/>
+<box size="0.3 0.3 0.2"/>
 </geometry>
 <origin xyz="0 0 0" rpy="0 0 0"/>
@@ -16,6 +17,8 @@
 <inertial>
 <origin xyz="0 0 0" rpy="0 0 0"/>
+<mass value="0.5"/>
 <inertia ixx="0.1" ixy="0.0" ixz="0.0" iyy="0.1" iyz="0.0" izz="0.1"/>
 </inertial>
 </link>
+</xacro:macro>
 </robot>

File: kodlar/kado.urdf (robot description, URDF)
Before this commit: robot roboke, 13 links, 12 joints
Links:
- link base_link: geometry collision cylinder length=0.08 radius=0.1; visual mesh filename=/home/samet/Desktop/isaac_robomaster/meshes/stl/mecanummain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 scale=0.002 0.002 0.002
- link mcn1: geometry collision mesh filename=/home/samet/Desktop/isaac_robomaster/meshes/stl/mecanumroll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 scale=0.002 0.002 0.002; visual mesh filename=/home/samet/Desktop/isaac_robomaster/meshes/stl/mecanumroll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 scale=0.002 0.002 0.002
- link mcn10: geometry collision mesh filename=/home/samet/Desktop/isaac_robomaster/meshes/stl/mecanumroll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 scale=0.002 0.002 0.002; visual mesh filename=/home/samet/Desktop/isaac_robomaster/meshes/stl/mecanumroll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 scale=0.002 0.002 0.002
- link mcn11: geometry collision mesh filename=/home/samet/Desktop/isaac_robomaster/meshes/stl/mecanumroll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 scale=0.002 0.002 0.002; visual mesh filename=/home/samet/Desktop/isaac_robomaster/meshes/stl/mecanumroll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 scale=0.002 0.002 0.002
- link mcn12: geometry collision mesh filename=/home/samet/Desktop/isaac_robomaster/meshes/stl/mecanumroll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 scale=0.002 0.002 0.002; visual mesh filename=/home/samet/Desktop/isaac_robomaster/meshes/stl/mecanumroll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 scale=0.002 0.002 0.002
- link mcn2: geometry collision mesh filename=/home/samet/Desktop/isaac_robomaster/meshes/stl/mecanumroll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 scale=0.002 0.002 0.002; visual mesh filename=/home/samet/Desktop/isaac_robomaster/meshes/stl/mecanumroll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 scale=0.002 0.002 0.002
- link mcn3: geometry collision mesh filename=/home/samet/Desktop/isaac_robomaster/meshes/stl/mecanumroll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 scale=0.002 0.002 0.002; visual mesh filename=/home/samet/Desktop/isaac_robomaster/meshes/stl/mecanumroll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 scale=0.002 0.002 0.002
- link mcn4: geometry collision mesh filename=/home/samet/Desktop/isaac_robomaster/meshes/stl/mecanumroll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 scale=0.002 0.002 0.002; visual mesh filename=/home/samet/Desktop/isaac_robomaster/meshes/stl/mecanumroll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 scale=0.002 0.002 0.002
- link mcn5: geometry collision mesh filename=/home/samet/Desktop/isaac_robomaster/meshes/stl/mecanumroll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 scale=0.002 0.002 0.002; visual mesh filename=/home/samet/Desktop/isaac_robomaster/meshes/stl/mecanumroll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 scale=0.002 0.002 0.002
- link mcn6: geometry collision mesh filename=/home/samet/Desktop/isaac_robomaster/meshes/stl/mecanumroll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 scale=0.002 0.002 0.002; visual mesh filename=/home/samet/Desktop/isaac_robomaster/meshes/stl/mecanumroll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 scale=0.002 0.002 0.002
- link mcn7: geometry collision mesh filename=/home/samet/Desktop/isaac_robomaster/meshes/stl/mecanumroll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 scale=0.002 0.002 0.002; visual mesh filename=/home/samet/Desktop/isaac_robomaster/meshes/stl/mecanumroll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 scale=0.002 0.002 0.002
- link mcn8: geometry collision mesh filename=/home/samet/Desktop/isaac_robomaster/meshes/stl/mecanumroll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 scale=0.002 0.002 0.002; visual mesh filename=/home/samet/Desktop/isaac_robomaster/meshes/stl/mecanumroll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 scale=0.002 0.002 0.002
- link mcn9: geometry collision mesh filename=/home/samet/Desktop/isaac_robomaster/meshes/stl/mecanumroll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 scale=0.002 0.002 0.002; visual mesh filename=/home/samet/Desktop/isaac_robomaster/meshes/stl/mecanumroll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 scale=0.002 0.002 0.002

File: kodlar/test.urdf.xacro (robot description, xacro)
@@ -1,5 +1,37 @@
 <?xml version="1.0"?>
 <robot name="roboke" xmlns:xacro="http://www.ros.org/wiki/xacro">
-<xacro:include filename="/home/samet/Desktop/robomaster-stl-files/wheels/kodlar/robomas.urdf.xacro"/>
+<xacro:include filename="/home/samet/Desktop/robomaster-stl-files/wheels/kodlar/arkatekerler/omnihazirL.xacro"/>
+<xacro:include filename="/home/samet/Desktop/robomaster-stl-files/wheels/kodlar/arkatekerler/omnihazirR.xacro"/>
+<xacro:include filename="/home/samet/Desktop/robomaster-stl-files/wheels/kodlar/arkatekerler/arkahazirL.xacro"/>
+<xacro:include filename="/home/samet/Desktop/robomaster-stl-files/wheels/kodlar/arkatekerler/arkahazirR.xacro"/>
+<xacro:include filename="/home/samet/Desktop/robomaster-stl-files/wheels/kodlar/chasishazir.xacro"/>
 <xacro:leko/>
+<xacro:leko2/>
+<xacro:leko3/>
+<xacro:leko4/>
+<joint name="joint_name2" type="continuous">
+    <parent link="basee_link"/>
+    <child link="base_link"/>
+    <axis xyz="0 0 1"/>
+    <origin xyz="0 0 0" rpy="0 0 0"/>
+</joint>
+<joint name="joint_name3" type="continuous">
+    <parent link="basee_link"/>
+    <child link="base_link2"/>
+    <axis xyz="0 0 1"/>
+    <origin xyz="0 0 0" rpy="0 0 0"/>
+</joint>
+<joint name="joint_name4" type="continuous">
+    <parent link="basee_link"/>
+    <child link="base_link3"/>
+    <axis xyz="0 0 1"/>
+    <origin xyz="0 0 0" rpy="0 0 0"/>
+</joint>
+<joint name="joint_name5" type="continuous">
+    <parent link="basee_link"/>
+    <child link="base_link4"/>
+    <axis xyz="0 0 1"/>
+    <origin xyz="0 0 0" rpy="0 0 0"/>
+</joint>
+<xacro:chasis/>
 </robot>
